File: customESC.sch (EAGLE design)
At the start: 7 parts

Commit message: Made some progress on schematic
Parts:
- added C1, C11, C13, C15, C17, C19, C21, C23, C3, C5, C7, C9: 10uF, SparkFun-Capacitors:10UF-0603-6.3V-20%
- added C10, C12, C14, C16, C18, C2, C20, C22, C24, C4, C6, C8: 2.2uF, SparkFun-Capacitors:10UF-0603-6.3V-20%
- added CONN1: 12V-CONNECTOR, X15-CustomESC:12V-CONNECTOR
- added D10, D11, D12, D13, D14, D3, D4, D5, D6, D7, D8, D9: IN4148WS, X15-CustomESC:IN4148WS
- added DRIV1, DRIV10, DRIV11, DRIV12, DRIV2, DRIV3, DRIV4, DRIV5, DRIV6, DRIV7, DRIV8, DRIV9: IR2101STRPBF, X15-CustomESC:IR2101STRPBF
- added H1, H2, H3, H4: 6-32-HOLE, X15-CustomESC:6-32-HOLE
- added MOS1, MOS10, MOS11, MOS12, MOS13, MOS14, MOS15, MOS16, MOS17, MOS18, MOS19, MOS2, MOS20, MOS21, MOS22, MOS23, MOS24, MOS3, MOS4, MOS5, MOS6, MOS7, MOS8, MOS9: IRLR7843TRPBF, X15-CustomESC:IRLR7843TRPBF
- added OUT1, OUT2, OUT3, OUT4: IPBT-103-H1-T-S, X15-CustomESC:IPBT-103-H1-T-S
- added R10, R11, R12, R13, R14, R15, R16, R17, R18, R19, R20, R21, R22, R23, R24, R25, R26, R3, R4, R5, R6, R7, R8, R9: 100, SparkFun-Resistors:1KOHM-0603-1/10W-1%
- added U$1: STM32F042K6T6, X15-CustomESC:STM32F042K6T6
- added U$2: JST_8_PIN, X15-CustomESC:JST_8_PIN
Connections:
- new net ADC: U$2.ADC
- new net AH1: DRIV1.HIN
- new net AH2: DRIV4.HIN
- new net AH3: DRIV7.HIN
- new net AH4: DRIV10.HIN
- new net AL1: DRIV1.!LIN
- new net AL2: DRIV4.!LIN
- new net AL3: DRIV7.!LIN
- new net AL4: DRIV10.!LIN
- new net BH1: DRIV2.HIN
- new net BH2: DRIV5.HIN
- new net BH3: DRIV8.HIN
- new net BH4: DRIV11.HIN
- new net BL1: DRIV2.!LIN
- new net BL2: DRIV5.!LIN
- new net BL3: DRIV8.!LIN
- new net BL4: DRIV11.!LIN
- new net CH1: DRIV3.HIN
- new net CH2: DRIV6.HIN
- new net CH3: DRIV9.HIN
- new net CH4: DRIV12.HIN
- new net CL1: DRIV3.!LIN
- new net CL2: DRIV6.!LIN
- new net CL3: DRIV9.!LIN
- new net CL4: DRIV12.!LIN
- new net LIPO_GND: U$2.LIPO_GND
- new net LIPO_IN: U$2.LIPO_IN
- new net N$10: DRIV2.LO, R6.1
- new net N$11: MOS3.GATE, R5.2
- new net N$12: MOS4.GATE, R6.2
- new net N$13: C6.1, D5.P$2, DRIV3.VB
- new net N$14: DRIV3.HO, R7.1
- new net N$15: DRIV3.LO, R8.1
- new net N$16: MOS5.GATE, R7.2
- new net N$17: MOS6.GATE, R8.2
- new net N$18: C8.1, D6.P$2, DRIV4.VB
- new net N$19: DRIV4.HO, R9.1
- new net N$20: DRIV4.LO, R10.1
- new net N$21: MOS7.GATE, R9.2
- new net N$22: MOS8.GATE, R10.2
- new net N$23: C10.1, D7.P$2, DRIV5.VB
- new net N$24: DRIV5.HO, R11.1
- new net N$25: DRIV5.LO, R12.1
- new net N$26: MOS9.GATE, R11.2
- new net N$27: MOS10.GATE, R12.2
- new net N$28: C12.1, D8.P$2, DRIV6.VB
- new net N$29: DRIV6.HO, R13.1
- new net N$3: C2.1, D3.P$2, DRIV1.VB
- new net N$30: DRIV6.LO, R14.1
- new net N$31: MOS11.GATE, R13.2
- new net N$32: MOS12.GATE, R14.2
- new net N$33: C14.1, D9.P$2, DRIV7.VB
- new net N$34: DRIV7.HO, R15.1
- new net N$35: DRIV7.LO, R16.1
- new net N$36: MOS13.GATE, R15.2
- new net N$37: MOS14.GATE, R16.2
- new net N$38: C16.1, D10.P$2, DRIV8.VB
- new net N$39: DRIV8.HO, R17.1
- new net N$4: DRIV1.HO, R3.1
- new net N$40: DRIV8.LO, R18.1
- new net N$41: MOS15.GATE, R17.2
- new net N$42: MOS16.GATE, R18.2
- new net N$43: C18.1, D11.P$2, DRIV9.VB
- new net N$44: DRIV9.HO, R19.1
- new net N$45: DRIV9.LO, R20.1
- new net N$46: MOS17.GATE, R19.2
- new net N$47: MOS18.GATE, R20.2
- new net N$48: C20.1, D12.P$2, DRIV10.VB
- new net N$49: DRIV10.HO, R21.1
- new net N$5: MOS1.GATE, R3.2
- new net N$50: DRIV10.LO, R22.1
- new net N$51: MOS19.GATE, R21.2
- new net N$52: MOS20.GATE, R22.2
- new net N$53: C22.1, D13.P$2, DRIV11.VB
- new net N$54: DRIV11.HO, R23.1
- new net N$55: DRIV11.LO, R24.1
- new net N$56: MOS21.GATE, R23.2
- new net N$57: MOS22.GATE, R24.2
- new net N$58: C24.1, D14.P$2, DRIV12.VB
- new net N$59: DRIV12.HO, R25.1
- new net N$6: DRIV1.LO, R4.1
- new net N$60: DRIV12.LO, R26.1
- new net N$61: MOS23.GATE, R25.2
- new net N$62: MOS24.GATE, R26.2
- new net N$7: MOS2.GATE, R4.2
- new net N$8: C4.1, D4.P$2, DRIV2.VB
- new net N$9: DRIV2.HO, R5.1
- new net PHASE_A1: C2.2, DRIV1.VS, MOS1.DRAIN, MOS2.SOURCE, OUT1.A
- new net PHASE_A2: C8.2, DRIV4.VS, MOS7.DRAIN, MOS8.SOURCE, OUT2.A
- new net PHASE_A3: C14.2, DRIV7.VS, MOS13.DRAIN, MOS14.SOURCE, OUT3.A
- new net PHASE_A4: C20.2, DRIV10.VS, MOS19.DRAIN, MOS20.SOURCE, OUT4.A
- new net PHASE_B1: C4.2, DRIV2.VS, MOS3.DRAIN, MOS4.SOURCE, OUT1.B
- new net PHASE_B2: C10.2, DRIV5.VS, MOS10.SOURCE, MOS9.DRAIN, OUT2.B
- new net PHASE_B3: C16.2, DRIV8.VS, MOS15.DRAIN, MOS16.SOURCE, OUT3.B
- new net PHASE_B4: C22.2, DRIV11.VS, MOS21.DRAIN, MOS22.SOURCE, OUT4.B
- new net PHASE_C1: C6.2, DRIV3.VS, MOS5.DRAIN, MOS6.SOURCE, OUT1.C
- new net PHASE_C2: C12.2, DRIV6.VS, MOS11.DRAIN, MOS12.SOURCE, OUT2.C
- new net PHASE_C3: C18.2, DRIV9.VS, MOS17.DRAIN, MOS18.SOURCE, OUT3.C
- new net PHASE_C4: C24.2, DRIV12.VS, MOS23.DRAIN, MOS24.SOURCE, OUT4.C
- new net TIM1: U$2.MTR_1
- new net TIM2: U$2.MTR_2
- new net TIM3: U$2.MTR_3
- new net TIM4: U$2.MTR_4
- new net TLM: U$2.TLM
- net GND: now also C1.2, C11.2, C13.2, C15.2, C17.2, C19.2, C21.2, C23.2, C3.2, C5.2, C7.2, C9.2, CONN1.GND, DRIV1.COM, DRIV10.COM, DRIV11.COM, DRIV12.COM, DRIV2.COM, DRIV3.COM, DRIV4.COM, DRIV5.COM, DRIV6.COM, DRIV7.COM, DRIV8.COM, DRIV9.COM, MOS10.DRAIN, MOS12.DRAIN, MOS14.DRAIN, MOS16.DRAIN, MOS18.DRAIN, MOS2.DRAIN, MOS20.DRAIN, MOS22.DRAIN, MOS24.DRAIN, MOS4.DRAIN, MOS6.DRAIN, MOS8.DRAIN
- net VCC_2: now also C1.1, C11.1, C13.1, C15.1, C17.1, C19.1, C21.1, C23.1, C3.1, C5.1, C7.1, C9.1, CONN1.12V, D10.P$1, D11.P$1, D12.P$1, D13.P$1, D14.P$1, D3.P$1, D4.P$1, D5.P$1, D6.P$1, D7.P$1, D8.P$1, D9.P$1, DRIV1.VCC, DRIV10.VCC, DRIV11.VCC, DRIV12.VCC, DRIV2.VCC, DRIV3.VCC, DRIV4.VCC, DRIV5.VCC, DRIV6.VCC, DRIV7.VCC, DRIV8.VCC, DRIV9.VCC, MOS1.SOURCE, MOS11.SOURCE, MOS13.SOURCE, MOS15.SOURCE, MOS17.SOURCE, MOS19.SOURCE, MOS21.SOURCE, MOS23.SOURCE, MOS3.SOURCE, MOS5.SOURCE, MOS7.SOURCE, MOS9.SOURCE
Other:
- note added: "First Half"
- note added: "Motor 1"
- note added: "Motor 2"
- note added: "Motor 3"
- note added: "Motor 4"
- note added: "Motor Output"
- note added: "Power Inputs"
- note added: "STM32"
- note added: "Second Half"
- note added: "Three Phase switching bridge"
- note added: "might add a second one"

Commit message: Ready for design review? not really
Parts:
- added C25: 0.1uF, SparkFun-Capacitors:10UF-0603-6.3V-20%
- added C26: 4.7uF, SparkFun-Capacitors:10UF-0603-6.3V-20%
- added R27: 1k, SparkFun-Resistors:1KOHM-0603-1/10W-1%
- added S1: MOMENTARY-SWITCH-SPST-SMD-6.0X3.5MM, SparkFun-Switches:MOMENTARY-SWITCH-SPST-SMD-6.0X3.5MM
Connections:
- new net N$63: C25.1, R27.1, S1.2, U$1.NRST
- net GND: now also C25.2, C26.2, S1.1, U$1.BOOT0, U$1.VDDIO2, U$1.VSS
- net VCC_1: now also C26.1, R27.2, U$1.VDD, U$1.VDDA
Other:
- note added: "decoupling"
Changed lines of the file:
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@@
 <part name="U$2" library="X15-CustomESC" deviceset="JST_8_PIN" device=""/>
 <part name="FRAME4" library="SparkFun-Aesthetics" library_urn="urn:adsk.eagle:library:507" deviceset="FRAME-A4L" device=""/>
+<part name="SUPPLY70" library="SparkFun-PowerSymbols" library_urn="urn:adsk.eagle:library:530" deviceset="VCC_1" device="" value="3.3V"/>
+<part name="SUPPLY71" library="supply2" library_urn="urn:adsk.eagle:library:372" deviceset="GND" device=""/>
+<part name="SUPPLY72" library="supply2" library_urn="urn:adsk.eagle:library:372" deviceset="GND" device=""/>
+<part name="SUPPLY73" library="SparkFun-PowerSymbols" library_urn="urn:adsk.eagle:library:530" deviceset="VCC_1" device="" value="3.3V"/>
+<part name="C25" library="SparkFun-Capacitors" library_urn="urn:adsk.eagle:library:510" deviceset="10UF" device="-0603-6.3V-20%" package3d_urn="urn:adsk.eagle:package:37414/1" value="0.1uF"/>
+<part name="S1" library="SparkFun-Switches" library_urn="urn:adsk.eagle:library:535" deviceset="MOMENTARY-SWITCH-SPST" device="-SMD-6.0X3.5MM" package3d_urn="urn:adsk.eagle:package:40165/1"/>
+<part name="SUPPLY74" library="supply2" library_urn="urn:adsk.eagle:library:372" deviceset="GND" device=""/>
+<part name="R27" library="SparkFun-Resistors" library_urn="urn:adsk.eagle:library:532" deviceset="1KOHM" device="-0603-1/10W-1%" package3d_urn="urn:adsk.eagle:package:39650/1" value="1k"/>
+<part name="SUPPLY75" library="SparkFun-PowerSymbols" library_urn="urn:adsk.eagle:library:530" deviceset="VCC_1" device="" value="3.3V"/>
+<part name="C26" library="SparkFun-Capacitors" library_urn="urn:adsk.eagle:library:510" deviceset="10UF" device="-0603-6.3V-20%" package3d_urn="urn:adsk.eagle:package:37414/1" value="4.7uF"/>
+<part name="SUPPLY76" library="supply2" library_urn="urn:adsk.eagle:library:372" deviceset="GND" device=""/>
+<part name="SUPPLY77" library="SparkFun-PowerSymbols" library_urn="urn:adsk.eagle:library:530" deviceset="VCC_1" device="" value="3.3V"/>
 </parts>
 <sheets>
@@
 <text x="62.23" y="90.17" size="5.08" layer="91">STM32</text>
 <text x="106.68" y="53.34" size="1.27" layer="91">might add a second one</text>
+<text x="144.78" y="127" size="1.27" layer="91">decoupling</text>
 </plain>
 <instances>
@@
 <attribute name="NAME" x="128.27" y="156.21" size="1.778" layer="95"/>
 </instance>
+<instance part="SUPPLY70" gate="G$2" x="25.4" y="67.31" smashed="yes">
+<attribute name="VALUE" x="25.4" y="70.104" size="1.778" layer="96" align="bottom-center"/>
+</instance>
+<instance part="SUPPLY71" gate="GND" x="35.56" y="74.93" smashed="yes">
+<attribute name="VALUE" x="33.655" y="71.755" size="1.778" layer="96"/>
+</instance>
+<instance part="SUPPLY72" gate="GND" x="95.25" y="21.59" smashed="yes">
+<attribute name="VALUE" x="93.345" y="18.415" size="1.778" layer="96"/>
+</instance>
+<instance part="SUPPLY73" gate="G$2" x="25.4" y="43.18" smashed="yes">
+<attribute name="VALUE" x="25.4" y="45.974" size="1.778" layer="96" align="bottom-center"/>
+</instance>
+<instance part="C25" gate="G$1" x="11.43" y="40.894" smashed="yes">
+<attribute name="NAME" x="12.954" y="43.815" size="1.778" layer="95" font="vector"/>
+<attribute name="VALUE" x="12.954" y="38.735" size="1.524" layer="96" font="vector"/>
+</instance>
+<instance part="S1" gate="G$1" x="21.59" y="43.18" smashed="yes" rot="R90">
+<attribute name="NAME" x="20.066" y="43.18" size="1.778" layer="95" font="vector" rot="R90" align="bottom-center"/>
+</instance>
+<instance part="SUPPLY74" gate="GND" x="11.43" y="26.67" smashed="yes">
+<attribute name="VALUE" x="9.525" y="23.495" size="1.778" layer="96"/>
+</instance>
+<instance part="R27" gate="G$1" x="11.43" y="57.15" smashed="yes" rot="R90">
+<attribute name="NAME" x="9.906" y="57.15" size="1.778" layer="95" font="vector" rot="R90" align="bottom-center"/>
+<attribute name="VALUE" x="12.954" y="57.15" size="1.778" layer="96" font="vector" rot="R90" align="top-center"/>
+</instance>
+<instance part="SUPPLY75" gate="G$2" x="11.43" y="67.31" smashed="yes">
+<attribute name="VALUE" x="11.43" y="70.104" size="1.778" layer="96" align="bottom-center"/>
+</instance>
+<instance part="C26" gate="G$1" x="148.59" y="114.554" smashed="yes">
+<attribute name="NAME" x="150.114" y="117.475" size="1.778" layer="95" font="vector"/>
+<attribute name="VALUE" x="150.114" y="112.395" size="1.524" layer="96" font="vector"/>
+</instance>
+<instance part="SUPPLY76" gate="GND" x="148.59" y="106.68" smashed="yes">
+<attribute name="VALUE" x="146.685" y="103.505" size="1.778" layer="96"/>
+</instance>
+<instance part="SUPPLY77" gate="G$2" x="148.59" y="121.92" smashed="yes">
+<attribute name="VALUE" x="148.59" y="124.714" size="1.778" layer="96" align="bottom-center"/>
+</instance>
 </instances>
 <busses>
@@
 <wire x1="33.02" y1="116.84" x2="38.1" y2="116.84" width="0.1524" layer="91"/>
 </segment>
+<segment>
+<pinref part="U$1" gate="G$1" pin="VDD"/>
+<wire x1="30.48" y1="63.5" x2="25.4" y2="63.5" width="0.1524" layer="91"/>
+<pinref part="SUPPLY70" gate="G$2" pin="VCC_1"/>
+<wire x1="25.4" y1="63.5" x2="25.4" y2="67.31" width="0.1524" layer="91"/>
+</segment>
+<segment>
+<pinref part="U$1" gate="G$1" pin="VDDA"/>
+<wire x1="30.48" y1="43.18" x2="25.4" y2="43.18" width="0.1524" layer="91"/>
+<pinref part="SUPPLY73" gate="G$2" pin="VCC_1"/>
+</segment>
+<segment>
+<pinref part="R27" gate="G$1" pin="2"/>
+<pinref part="SUPPLY75" gate="G$2" pin="VCC_1"/>
+<wire x1="11.43" y1="62.23" x2="11.43" y2="67.31" width="0.1524" layer="91"/>
+</segment>
+<segment>
+<pinref part="C26" gate="G$1" pin="1"/>
+<wire x1="148.59" y1="119.634" x2="148.59" y2="121.92" width="0.1524" layer="91"/>
+<pinref part="SUPPLY77" gate="G$2" pin="VCC_1"/>
+</segment>
 </net>
 <net name="VCC_2" class="0">
@@
 <pinref part="SUPPLY69" gate="GND" pin="GND"/>
 </segment>
+<segment>
+<pinref part="U$1" gate="G$1" pin="VSS"/>
+<wire x1="43.18" y1="76.2" x2="43.18" y2="78.74" width="0.1524" layer="91"/>
+<wire x1="43.18" y1="78.74" x2="35.56" y2="78.74" width="0.1524" layer="91"/>
+<wire x1="35.56" y1="78.74" x2="35.56" y2="77.47" width="0.1524" layer="91"/>
+<pinref part="SUPPLY71" gate="GND" pin="GND"/>
+<pinref part="U$1" gate="G$1" pin="BOOT0"/>
+<wire x1="48.26" y1="76.2" x2="48.26" y2="78.74" width="0.1524" layer="91"/>
+<wire x1="48.26" y1="78.74" x2="43.18" y2="78.74" width="0.1524" layer="91"/>
+<junction x="43.18" y="78.74"/>
+</segment>
+<segment>
+<pinref part="U$1" gate="G$1" pin="VDDIO2"/>
+<wire x1="91.44" y1="27.94" x2="95.25" y2="27.94" width="0.1524" layer="91"/>
+<wire x1="95.25" y1="27.94" x2="95.25" y2="24.13" width="0.1524" layer="91"/>
+<pinref part="SUPPLY72" gate="GND" pin="GND"/>
+</segment>
+<segment>
+<pinref part="C25" gate="G$1" pin="2"/>
+<wire x1="11.43" y1="38.354" x2="11.43" y2="31.75" width="0.1524" layer="91"/>
+<pinref part="S1" gate="G$1" pin="1"/>
+<wire x1="11.43" y1="31.75" x2="11.43" y2="29.21" width="0.1524" layer="91"/>
+<wire x1="21.59" y1="38.1" x2="21.59" y2="31.75" width="0.1524" layer="91"/>
+<wire x1="21.59" y1="31.75" x2="11.43" y2="31.75" width="0.1524" layer="91"/>
+<junction x="11.43" y="31.75"/>
+<pinref part="SUPPLY74" gate="GND" pin="GND"/>
+</segment>
+<segment>
+<pinref part="C26" gate="G$1" pin="2"/>
+<wire x1="148.59" y1="112.014" x2="148.59" y2="109.22" width="0.1524" layer="91"/>
+<pinref part="SUPPLY76" gate="GND" pin="GND"/>
+</segment>
 </net>
 <net name="PHASE_A1" class="0">
@@
 </segment>
 </net>
+<net name="N$63" class="0">
+<segment>
+<pinref part="U$1" gate="G$1" pin="NRST"/>
+<wire x1="30.48" y1="48.26" x2="21.59" y2="48.26" width="0.1524" layer="91"/>
+<pinref part="S1" gate="G$1" pin="2"/>
+<junction x="21.59" y="48.26"/>
+<pinref part="C25" gate="G$1" pin="1"/>
+<wire x1="21.59" y1="48.26" x2="11.43" y2="48.26" width="0.1524" layer="91"/>
+<wire x1="11.43" y1="48.26" x2="11.43" y2="45.974" width="0.1524" layer="91"/>
+<pinref part="R27" gate="G$1" pin="1"/>
+<wire x1="11.43" y1="48.26" x2="11.43" y2="52.07" width="0.1524" layer="91"/>
+<junction x="11.43" y="48.26"/>
+</segment>
+</net>
