File: customESC_Test_Board.sch (EAGLE design)
At the start: 54 parts

Commit message: Added a new file
Parts:
- added C10, C12, C14, C16, C18, C20, C22, C24, C8: 2.2uF, SparkFun-Capacitors:10UF-0603-6.3V-20%
- added C11, C13, C15, C17, C19, C21, C23, C7, C9: 10uF, SparkFun-Capacitors:10UF-0603-6.3V-20%
- added CNTRL: JST_8_PIN, X15-CustomESC:JST_8_PIN
- added D10, D11, D12, D13, D14, D6, D7, D8, D9: IN4148WS, X15-CustomESC:IN4148WS
- added DRIV10, DRIV11, DRIV12, DRIV4, DRIV5, DRIV6, DRIV7, DRIV8, DRIV9: IR2101STRPBF, X15-CustomESC:IR2101STRPBF
- added MOS10, MOS11, MOS12, MOS13, MOS14, MOS15, MOS16, MOS17, MOS18, MOS19, MOS20, MOS21, MOS22, MOS23, MOS24, MOS7, MOS8, MOS9: IRLR7843TRPBF, X15-CustomESC:IRLR7843TRPBF
- added OUT2, OUT3, OUT4: IPBT-103-H1-T-S, X15-CustomESC:IPBT-103-H1-T-S
- added R10, R11, R12, R13, R14, R15, R16, R17, R18, R19, R20, R21, R22, R23, R24, R25, R26, R9: 100, SparkFun-Resistors:1KOHM-0603-1/10W-1%
- added R40, R41, R42, R43, R44, R45, R49, R50, R51, R52, R53, R54, R55, R56, R57, R61, R62, R63, R64, R65, R66, R67, R68, R69, R73, R74, R75: 33k, SparkFun-Resistors:1KOHM-0603-1/10W-1%
- added R46, R47, R48, R58, R59, R60, R70, R71, R72: 10k, SparkFun-Resistors:1KOHM-0603-1/10W-1%
- added STM2: STM32F042K6T6, X15-CustomESC:STM32F042K6T6
Connections:
- new net ADC: CNTRL.ADC
- new net AH2: DRIV4.HIN, STM1.PA14
- new net AH3: DRIV7.HIN, STM2.PA8
- new net AH4: DRIV10.HIN, STM2.PA14
- new net AL2: DRIV4.!LIN, STM1.PB4
- new net AL3: DRIV7.!LIN, STM2.PA11
- new net AL4: DRIV10.!LIN, STM2.PB4
- new net BEMF_A2: R61.2, STM1.PA5
- new net BEMF_A3: R49.2, STM2.PA2
- new net BEMF_A4: R73.2, STM2.PA5
- new net BEMF_B2: R62.2, STM1.PA6
- new net BEMF_B3: R50.2, STM2.PA3
- new net BEMF_B4: R74.2, STM2.PA6
- new net BEMF_C2: R63.2, STM1.PA7
- new net BEMF_C3: R51.2, STM2.PA4
- new net BEMF_C4: R75.2, STM2.PA7
- new net BH2: DRIV5.HIN, STM1.PA15
- new net BH3: DRIV8.HIN, STM2.PA9
- new net BH4: DRIV11.HIN, STM2.PA15
- new net BL2: DRIV5.!LIN, STM1.PB5
- new net BL3: DRIV8.!LIN, STM2.PA12
- new net BL4: DRIV11.!LIN, STM2.PB5
- new net CH2: DRIV6.HIN, STM1.PB3
- new net CH3: DRIV9.HIN, STM2.PA10
- new net CH4: DRIV12.HIN, STM2.PB3
- new net CL2: DRIV6.!LIN, STM1.PB6
- new net CL3: DRIV9.!LIN, STM2.PA13
- new net CL4: DRIV12.!LIN, STM2.PB6
- new net COM2: R52.1, R53.1, R54.1, STM1.PA1
- new net COM3: R40.1, R41.1, R42.1, STM2.PA0
- new net COM4: R64.1, R65.1, R66.1, STM2.PA1
- new net LIPO_GND: CNTRL.LIPO_GND
- new net LIPO_IN: CNTRL.LIPO_IN
- new net N$19: DRIV4.HO, R9.1
- new net N$20: DRIV4.LO, R10.1
- new net N$21: MOS7.GATE, R9.2
- new net N$22: MOS8.GATE, R10.2
- new net N$23: C10.1, D7.P$2, DRIV5.VB
- new net N$24: DRIV5.HO, R11.1
- new net N$25: DRIV5.LO, R12.1
- new net N$26: MOS9.GATE, R11.2
- new net N$27: MOS10.GATE, R12.2
- new net N$28: C12.1, D8.P$2, DRIV6.VB
- new net N$29: DRIV6.HO, R13.1
- new net N$30: DRIV6.LO, R14.1
- new net N$31: MOS11.GATE, R13.2
- new net N$32: MOS12.GATE, R14.2
- new net N$33: C14.1, D9.P$2, DRIV7.VB
- new net N$34: DRIV7.HO, R15.1
- new net N$35: DRIV7.LO, R16.1
- new net N$36: MOS13.GATE, R15.2
- new net N$37: MOS14.GATE, R16.2
- new net N$38: C16.1, D10.P$2, DRIV8.VB
- new net N$39: DRIV8.HO, R17.1
- new net N$40: DRIV8.LO, R18.1
- new net N$41: MOS15.GATE, R17.2
- new net N$42: MOS16.GATE, R18.2
- new net N$43: C18.1, D11.P$2, DRIV9.VB
- new net N$44: DRIV9.HO, R19.1
- new net N$45: DRIV9.LO, R20.1
- new net N$46: MOS17.GATE, R19.2
- new net N$47: MOS18.GATE, R20.2
- new net N$48: C20.1, D12.P$2, DRIV10.VB
- new net N$49: DRIV10.HO, R21.1
- new net N$50: DRIV10.LO, R22.1
- new net N$51: MOS19.GATE, R21.2
- new net N$52: MOS20.GATE, R22.2
- new net N$53: C22.1, D13.P$2, DRIV11.VB
- new net N$54: DRIV11.HO, R23.1
- new net N$55: DRIV11.LO, R24.1
- new net N$56: MOS21.GATE, R23.2
- new net N$57: MOS22.GATE, R24.2
- new net N$58: C24.1, D14.P$2, DRIV12.VB
- new net N$59: DRIV12.HO, R25.1
- new net N$60: DRIV12.LO, R26.1
- new net N$61: MOS23.GATE, R25.2
- new net N$62: MOS24.GATE, R26.2
- new net N$67: R40.2, R43.1, R46.2, R49.1
- new net N$68: R41.2, R44.1, R47.2, R50.1
- new net N$69: R42.2, R45.1, R48.2, R51.1
- new net N$70: R52.2, R55.1, R58.2, R61.1
- new net N$71: R53.2, R56.1, R59.2, R62.1
- new net N$72: R54.2, R57.1, R60.2, R63.1
- new net N$73: R64.2, R67.1, R70.2, R73.1
- new net N$74: R65.2, R68.1, R71.2, R74.1
- new net N$75: R66.2, R69.1, R72.2, R75.1
- new net PHASE_A2: C8.2, DRIV4.VS, MOS7.DRAIN, MOS8.SOURCE, OUT2.A, R55.2
- new net PHASE_A3: C14.2, DRIV7.VS, MOS13.DRAIN, MOS14.SOURCE, OUT3.A, R43.2
- new net PHASE_A4: C20.2, DRIV10.VS, MOS19.DRAIN, MOS20.SOURCE, OUT4.A, R67.2
- new net PHASE_B2: C10.2, DRIV5.VS, MOS10.SOURCE, MOS9.DRAIN, OUT2.B, R56.2
- new net PHASE_B3: C16.2, DRIV8.VS, MOS15.DRAIN, MOS16.SOURCE, OUT3.B, R44.2
- new net PHASE_B4: C22.2, DRIV11.VS, MOS21.DRAIN, MOS22.SOURCE, OUT4.B, R68.2
- new net PHASE_C2: C12.2, DRIV6.VS, MOS11.DRAIN, MOS12.SOURCE, OUT2.C, R57.2
- new net PHASE_C3: C18.2, DRIV9.VS, MOS17.DRAIN, MOS18.SOURCE, OUT3.C, R45.2
- new net PHASE_C4: C24.2, DRIV12.VS, MOS23.DRAIN, MOS24.SOURCE, OUT4.C, R69.2
- new net TIM2: CNTRL.MTR_2, STM1.PB1
- new net TIM3: CNTRL.MTR_3, STM2.PB0
- new net TIM4: CNTRL.MTR_4, STM2.PB1
- new net TLM: CNTRL.TLM
- net GND: now also C11.2, C13.2, C15.2, C17.2, C19.2, C21.2, C23.2, C7.2, C9.2, DRIV10.COM, DRIV11.COM, DRIV12.COM, DRIV4.COM, DRIV5.COM, DRIV6.COM, DRIV7.COM, DRIV8.COM, DRIV9.COM, MOS10.DRAIN, MOS12.DRAIN, MOS14.DRAIN, MOS16.DRAIN, MOS18.DRAIN, MOS20.DRAIN, MOS22.DRAIN, MOS24.DRAIN, MOS8.DRAIN, R46.1, R47.1, R48.1, R58.1, R59.1, R60.1, R70.1, R71.1, R72.1, STM2.PB8, STM2.VDDIO2, STM2.VSS
- net N$18: now also C8.1, D6.P$2, DRIV4.VB; no longer STM1.PA6
- net NRST: now also STM2.NRST
- net TIM1: now also CNTRL.MTR_1
- net VCC_1: now also STM2.VDD, STM2.VDDA
- net VCC_2: now also C11.1, C13.1, C15.1, C17.1, C19.1, C21.1, C23.1, C7.1, C9.1, D10.P$1, D11.P$1, D12.P$1, D13.P$1, D14.P$1, D6.P$1, D7.P$1, D8.P$1, D9.P$1, DRIV10.VCC, DRIV11.VCC, DRIV12.VCC, DRIV4.VCC, DRIV5.VCC, DRIV6.VCC, DRIV7.VCC, DRIV8.VCC, DRIV9.VCC, MOS11.SOURCE, MOS13.SOURCE, MOS15.SOURCE, MOS17.SOURCE, MOS19.SOURCE, MOS21.SOURCE, MOS23.SOURCE, MOS7.SOURCE, MOS9.SOURCE
Other:
- note added: "Control Inputs"
- note added: "First Half"
- note added: "Motor 2"
- note added: "Motor 3"
- note added: "Motor 4"
- note added: "Second Half"
