File: customESC_Test.sch (EAGLE design)
At the start: 54 parts

Commit message: update
lol
Connections:
- net N$13 renamed VB_3
- net N$3 renamed VB_1
- net N$8 renamed VB_2
Changed lines of the file:
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@@
 </segment>
 </net>
-<net name="N$3" class="0">
+<net name="VB_1" class="0">
 <segment>
 <pinref part="D3" gate="G$1" pin="P$2"/>
@@
 <wire x1="77.47" y1="139.7" x2="77.47" y2="151.13" width="0.1524" layer="91"/>
 <junction x="77.47" y="151.13"/>
+<label x="74.93" y="146.05" size="1.778" layer="95"/>
 </segment>
 </net>
@@
 </segment>
 </net>
-<net name="N$8" class="0">
+<net name="VB_2" class="0">
 <segment>
 <pinref part="D4" gate="G$1" pin="P$2"/>
@@
 <wire x1="78.74" y1="99.06" x2="78.74" y2="110.49" width="0.1524" layer="91"/>
 <junction x="78.74" y="110.49"/>
+<label x="74.93" y="105.41" size="1.778" layer="95"/>
 </segment>
 </net>
@@
 </segment>
 </net>
-<net name="N$13" class="0">
-<segment>
-<pinref part="D5" gate="G$1" pin="P$2"/>
-<pinref part="C6" gate="G$1" pin="1"/>
-<wire x1="69.596" y1="67.31" x2="78.74" y2="67.31" width="0.1524" layer="91"/>
-<pinref part="DRIV3" gate="DRV$1" pin="VB"/>
-<wire x1="78.74" y1="67.31" x2="85.09" y2="67.31" width="0.1524" layer="91"/>
-<wire x1="77.47" y1="55.88" x2="78.74" y2="55.88" width="0.1524" layer="91"/>
-<wire x1="78.74" y1="55.88" x2="78.74" y2="67.31" width="0.1524" layer="91"/>
-<junction x="78.74" y="67.31"/>
-</segment>
-</net>
 <net name="N$14" class="0">
 <segment>
@@
 </segment>
 </net>
+<net name="VB_3" class="0">
+<segment>
+<pinref part="D5" gate="G$1" pin="P$2"/>
+<pinref part="C6" gate="G$1" pin="1"/>
+<wire x1="69.596" y1="67.31" x2="78.74" y2="67.31" width="0.1524" layer="91"/>
+<pinref part="DRIV3" gate="DRV$1" pin="VB"/>
+<wire x1="78.74" y1="67.31" x2="85.09" y2="67.31" width="0.1524" layer="91"/>
+<wire x1="77.47" y1="55.88" x2="78.74" y2="55.88" width="0.1524" layer="91"/>
+<wire x1="78.74" y1="55.88" x2="78.74" y2="67.31" width="0.1524" layer="91"/>
+<junction x="78.74" y="67.31"/>
+<label x="74.93" y="58.42" size="1.778" layer="95"/>
+</segment>
+</net>

Commit message: lol
Parts:
- added BLUE, GREEN, RED, YELLOW: (no value), led:LEDCHIPLED_0805
- added JP1: (no value), pinhead:PINHD-1X1
- added R9: (no value), pot:3RP/1610N
Connections:
- removed net N$18: STM1.PA6
- new net PWM_IN: JP1.1, R9.S, STM1.PA6
- new net TEST_LED1: RED.A, STM1.PB6
- new net TEST_LED2: BLUE.A, STM1.PB5
- new net TEST_LED3: STM1.PB4, YELLOW.A
- new net TEST_LED4: GREEN.A, STM1.PB3
- net GND: now also BLUE.C, GREEN.C, R9.A, RED.C, YELLOW.C
- net VCC_1: now also R9.E
Other:
- note added: "Potentiometer Input"
- note added: "Real PWM Input"

Commit message: done
Parts:
- added J1: 3V3 -SWCLK-GND-SWDIO- NRST, X15-ESC-Controller-Parts-Library:SWD_CONN
Connections:
- new net SWCLK: J1.SWCLK, STM1.PA14
- new net SWDIO: J1.SWDIO, STM1.PA15
- net GND: now also J1.GND
- net NRST: now also J1.NRST
- net VCC_1: now also J1.3V3
Other:
- note added: "USB_CON"
Changed lines of the file:
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@@
 <layer number="56" name="wert" color="7" fill="1" visible="no" active="no"/>
 <layer number="57" name="tCAD" color="7" fill="1" visible="no" active="no"/>
+<layer number="58" name="bCopper" color="7" fill="1" visible="no" active="no"/>
 <layer number="59" name="tCarbon" color="7" fill="1" visible="no" active="no"/>
 <layer number="60" name="bCarbon" color="7" fill="1" visible="no" active="no"/>
@@
 <layer number="115" name="ReferenceISLANDS" color="7" fill="1" visible="no" active="yes"/>
 <layer number="116" name="Patch_BOT" color="9" fill="4" visible="yes" active="yes"/>
+<layer number="117" name="PM_Ref" color="7" fill="1" visible="no" active="no"/>
 <layer number="118" name="Rect_Pads" color="7" fill="1" visible="no" active="yes"/>
+<layer number="119" name="PF_Ref" color="7" fill="1" visible="no" active="no"/>
+<layer number="120" name="WFL_Ref" color="7" fill="1" visible="no" active="no"/>
 <layer number="121" name="_tsilk" color="7" fill="1" visible="yes" active="yes"/>
 <layer number="122" name="_bsilk" color="7" fill="1" visible="yes" active="yes"/>
@@
 <layer number="128" name="_bValues" color="7" fill="1" visible="yes" active="yes"/>
 <layer number="129" name="Mask" color="7" fill="1" visible="yes" active="yes"/>
+<layer number="130" name="SMDSTROOK" color="7" fill="1" visible="no" active="no"/>
 <layer number="131" name="tAdjust" color="7" fill="1" visible="yes" active="yes"/>
 <layer number="132" name="bAdjust" color="7" fill="1" visible="yes" active="yes"/>
+<layer number="133" name="bottom_silk" color="7" fill="1" visible="no" active="no"/>
+<layer number="134" name="silk_top" color="7" fill="1" visible="no" active="no"/>
+<layer number="135" name="silk_bottom" color="7" fill="1" visible="no" active="no"/>
+<layer number="136" name="silktop" color="7" fill="1" visible="no" active="no"/>
+<layer number="137" name="silkbottom" color="7" fill="1" visible="no" active="no"/>
+<layer number="138" name="EEE" color="7" fill="1" visible="no" active="no"/>
+<layer number="139" name="_tKeepout" color="7" fill="1" visible="no" active="no"/>
+<layer number="140" name="mbKeepout" color="7" fill="1" visible="no" active="no"/>
+<layer number="141" name="ASSEMBLY_TOP" color="7" fill="1" visible="no" active="no"/>
+<layer number="142" name="mbRestrict" color="7" fill="1" visible="no" active="no"/>
+<layer number="143" name="PLACE_BOUND_TOP" color="7" fill="1" visible="no" active="no"/>
 <layer number="144" name="Drill_legend" color="7" fill="1" visible="yes" active="yes"/>
+<layer number="145" name="DrillLegend_01-02" color="7" fill="1" visible="no" active="no"/>
+<layer number="146" name="DrillLegend_01-15" color="7" fill="1" visible="no" active="no"/>
+<layer number="147" name="DrillLegend_01-16" color="7" fill="1" visible="no" active="no"/>
+<layer number="148" name="DrillLegend_01-20" color="7" fill="1" visible="no" active="no"/>
+<layer number="149" name="DrillLegend_02-15" color="7" fill="1" visible="no" active="no"/>
 <layer number="150" name="Notes" color="7" fill="1" visible="yes" active="yes"/>
 <layer number="151" name="HeatSink" color="7" fill="1" visible="yes" active="yes"/>
@@
 <layer number="154" name="FabDoc2" color="7" fill="1" visible="yes" active="yes"/>
 <layer number="155" name="FabDoc3" color="7" fill="1" visible="yes" active="yes"/>
+<layer number="156" name="gesam-Maß" color="7" fill="1" visible="no" active="no"/>
+<layer number="157" name="FaceMchng" color="7" fill="1" visible="no" active="no"/>
+<layer number="158" name="FaceMMeas" color="7" fill="1" visible="no" active="no"/>
+<layer number="159" name="Geh-Bear2" color="7" fill="1" visible="no" active="no"/>
+<layer number="160" name="Topologie" color="7" fill="1" visible="no" active="no"/>
+<layer number="161" name="tomplace2" color="7" fill="1" visible="no" active="no"/>
+<layer number="166" name="AntennaArea" color="7" fill="1" visible="no" active="no"/>
+<layer number="168" name="4mmHeightArea" color="7" fill="1" visible="no" active="no"/>
+<layer number="191" name="mNets" color="7" fill="1" visible="no" active="no"/>
+<layer number="192" name="mBusses" color="7" fill="1" visible="no" active="no"/>
+<layer number="193" name="mPins" color="7" fill="1" visible="no" active="no"/>
+<layer number="194" name="mSymbols" color="7" fill="1" visible="no" active="no"/>
+<layer number="195" name="mNames" color="7" fill="1" visible="no" active="no"/>
+<layer number="196" name="mValues" color="7" fill="1" visible="no" active="no"/>
 <layer number="199" name="Contour" color="7" fill="1" visible="yes" active="yes"/>
 <layer number="200" name="200bmp" color="1" fill="10" visible="yes" active="yes"/>
@@
 <layer number="250" name="Descript" color="3" fill="1" visible="no" active="no"/>
 <layer number="251" name="SMDround" color="12" fill="11" visible="no" active="no"/>
+<layer number="252" name="BR-BS" color="7" fill="1" visible="no" active="no"/>
+<layer number="253" name="Extra" color="7" fill="1" visible="no" active="no"/>
 <layer number="254" name="cooling" color="7" fill="1" visible="yes" active="yes"/>
 <layer number="255" name="routoute" color="7" fill="1" visible="yes" active="yes"/>
@@
 <part name="SUPPLY27" library="supply2" library_urn="urn:adsk.eagle:library:372" deviceset="GND" device=""/>
 <part name="SUPPLY28" library="supply2" library_urn="urn:adsk.eagle:library:372" deviceset="GND" device=""/>
+<part name="J1" library="X15-ESC-Controller-Parts-Library" deviceset="SWD_CONN" device="" value="3V3 -SWCLK-GND-SWDIO- NRST"/>
+<part name="SUPPLY29" library="SparkFun-PowerSymbols" library_urn="urn:adsk.eagle:library:530" deviceset="VCC_1" device="" value="3.3V"/>
 </parts>
 <sheets>
@@
 <text x="100.33" y="129.54" size="3.81" layer="91">Potentiometer Input</text>
 <text x="106.68" y="78.74" size="3.81" layer="91">Real PWM Input</text>
+<text x="158.75" y="109.22" size="3.81" layer="91">USB_CON</text>
 </plain>
 <instances>
@@
 <attribute name="VALUE" x="154.305" y="48.895" size="1.778" layer="96" rot="R180"/>
 </instance>
+<instance part="J1" gate="G$1" x="166.37" y="96.52" smashed="yes">
+<attribute name="NAME" x="158.75" y="104.648" size="1.778" layer="95" font="vector"/>
+</instance>
+<instance part="SUPPLY29" gate="G$2" x="186.69" y="104.14" smashed="yes">
+<attribute name="VALUE" x="186.69" y="106.934" size="1.778" layer="96" align="bottom-center"/>
+</instance>
 </instances>
 <busses>
@@
 <pinref part="R9" gate="G$1" pin="E"/>
 <wire x1="115.57" y1="118.11" x2="115.57" y2="114.3" width="0.1524" layer="91"/>
+</segment>
+<segment>
+<pinref part="J1" gate="G$1" pin="3V3"/>
+<wire x1="173.99" y1="101.6" x2="186.69" y2="101.6" width="0.1524" layer="91"/>
+<wire x1="186.69" y1="104.14" x2="186.69" y2="101.6" width="0.1524" layer="91"/>
+<pinref part="SUPPLY29" gate="G$2" pin="VCC_1"/>
 </segment>
 </net>
@@
 <pinref part="GREEN" gate="G$1" pin="C"/>
 <wire x1="152.4" y1="43.18" x2="152.4" y2="40.64" width="0.1524" layer="91"/>
+</segment>
+<segment>
+<pinref part="J1" gate="G$1" pin="GND"/>
+<wire x1="173.99" y1="96.52" x2="186.69" y2="96.52" width="0.1524" layer="91"/>
+<label x="184.15" y="96.52" size="1.778" layer="95" align="bottom-right"/>
 </segment>
 </net>
@@
 <label x="11.43" y="52.07" size="1.27" layer="95" rot="R180" xref="yes"/>
 </segment>
+<segment>
+<pinref part="J1" gate="G$1" pin="NRST"/>
+<wire x1="173.99" y1="91.44" x2="186.69" y2="91.44" width="0.1524" layer="91"/>
+<label x="184.15" y="91.44" size="1.778" layer="95" align="bottom-right"/>
+</segment>
 </net>
 <net name="COM1" class="0">
@@
 <wire x1="114.3" y1="33.02" x2="114.3" y2="31.75" width="0.1524" layer="91"/>
 <label x="114.3" y="31.75" size="1.778" layer="95" rot="R270" xref="yes"/>
+</segment>
+</net>
+<net name="SWDIO" class="0">
+<segment>
+<pinref part="J1" gate="G$1" pin="SWDIO"/>
+<wire x1="173.99" y1="93.98" x2="186.69" y2="93.98" width="0.1524" layer="91"/>
+<label x="184.15" y="93.98" size="1.778" layer="95" align="bottom-right"/>
+</segment>
+<segment>
+<pinref part="STM1" gate="G$1" pin="PA15"/>
+<wire x1="67.31" y1="80.01" x2="67.31" y2="81.28" width="0.1524" layer="91"/>
+<label x="67.31" y="81.28" size="1.778" layer="95" rot="R90" xref="yes"/>
+</segment>
+</net>
+<net name="SWCLK" class="0">
+<segment>
+<pinref part="J1" gate="G$1" pin="SWCLK"/>
+<wire x1="173.99" y1="99.06" x2="186.69" y2="99.06" width="0.1524" layer="91"/>
+<label x="184.15" y="99.06" size="1.778" layer="95" align="bottom-right"/>
+</segment>
+<segment>
+<pinref part="STM1" gate="G$1" pin="PA14"/>
+<wire x1="80.01" y1="67.31" x2="81.28" y2="67.31" width="0.1524" layer="91"/>
+<label x="81.28" y="67.31" size="1.778" layer="95" xref="yes"/>
 </segment>
 </net>
@@
 packages will not be understood (or retained) with this version.
 </note>
+<note version="9.0" severity="warning">
+Since Version 9.0, EAGLE supports the align property for labels.
+Labels in schematic will not be understood with this version. Update EAGLE to the latest version
+for full support of labels.
+</note>
 <note version="8.5" severity="warning">
