File: customESC_Test.sch (EAGLE design)
At the start: 61 parts, among them J1 3V3 -SWCLK-GND-SWDIO- NRST

Commit message: Fixed it Raghav
Hi
Connections:
- net PWM_IN: no longer R9.S
- net TIM1: now also R9.S
Changed lines of the file:
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@@
 <label x="57.15" y="17.78" size="1.27" layer="95" rot="R270" xref="yes"/>
+</segment>
+<segment>
+<pinref part="R9" gate="G$1" pin="S"/>
+<wire x1="120.65" y1="109.22" x2="123.19" y2="109.22" width="0.1524" layer="91"/>
+<label x="123.19" y="109.22" size="1.778" layer="95"/>
+<label x="123.19" y="109.22" size="1.778" layer="95"/>
 </segment>
 </net>
@@
 <net name="PWM_IN" class="0">
 <segment>
-<pinref part="R9" gate="G$1" pin="S"/>
-<wire x1="120.65" y1="109.22" x2="125.73" y2="109.22" width="0.1524" layer="91"/>
-<label x="125.73" y="109.22" size="1.778" layer="95"/>
-</segment>
-<segment>
 <pinref part="STM1" gate="G$1" pin="PA6"/>
