File: customESC_Test.brd (EAGLE design)
At the start: 152.4 x 127 mm, 61 parts, among them J1 3V3 -SWCLK-GND-SWDIO- NRST

Commit message: last one
Parts:
- moved J1 40.5 mm to (12.7, 19.1), turned to 90 degrees
Routing:
- net SWDIO: track 0.00 -> 90.6 mm, vias 0 -> 2
- net SWCLK: track 0.00 -> 88.7 mm, vias 0 -> 4
- net NRST: track 99.7 -> 146.6 mm
- net GND: track 272.2 -> 295.0 mm
- net VCC_1: track 263.7 -> 266.1 mm
Changed lines of the file:
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@@
 <attribute name="VALUE" x="102.87" y="119.38" size="1.27" layer="27" rot="R90"/>
 </element>
-<element name="J1" library="X15-ESC-Controller-Parts-Library" package="1X05" value="3V3 -SWCLK-GND-SWDIO- NRST" x="-13.97" y="-11.43" smashed="yes">
-<attribute name="NAME" x="-15.24" y="-10.033" size="0.6096" layer="25" font="vector" ratio="20"/>
-<attribute name="VALUE" x="-15.494" y="-13.716" size="0.6096" layer="25"/>
+<element name="J1" library="X15-ESC-Controller-Parts-Library" package="1X05" value="3V3 -SWCLK-GND-SWDIO- NRST" x="12.7" y="19.05" smashed="yes" rot="R90">
+<attribute name="NAME" x="11.303" y="17.78" size="0.6096" layer="25" font="vector" ratio="20" rot="R90"/>
+<attribute name="VALUE" x="14.986" y="17.526" size="0.6096" layer="25" rot="R90"/>
 </element>
 </elements>
@@
 <contactref element="R9" pad="3"/>
 <wire x1="48.34" y1="7.62" x2="44.53" y2="3.81" width="0.381" layer="1"/>
-<wire x1="44.53" y1="3.81" x2="19.05" y2="3.81" width="0.381" layer="1"/>
-<wire x1="19.05" y1="3.81" x2="16.51" y2="6.35" width="0.381" layer="1"/>
-<wire x1="16.51" y1="6.35" x2="16.51" y2="52.07" width="0.381" layer="1"/>
-<wire x1="16.51" y1="52.07" x2="25.26" y2="60.82" width="0.381" layer="1"/>
+<wire x1="44.53" y1="3.81" x2="27.94" y2="3.81" width="0.381" layer="1"/>
+<wire x1="27.94" y1="3.81" x2="20.32" y2="11.43" width="0.381" layer="1"/>
+<wire x1="20.32" y1="11.43" x2="20.32" y2="55.88" width="0.381" layer="1"/>
+<wire x1="20.32" y1="55.88" x2="25.26" y2="60.82" width="0.381" layer="1"/>
 <wire x1="25.26" y1="60.82" x2="49.53" y2="60.82" width="0.381" layer="1"/>
 <contactref element="J1" pad="1"/>
-<wire x1="30.48" y1="118.96" x2="34.837" y2="121.92" width="0" layer="19" extent="1-1"/>
-<wire x1="29.21" y1="124.46" x2="30.48" y2="118.96" width="0" layer="19" extent="1-1"/>
-<wire x1="24.13" y1="121.07" x2="29.21" y2="124.46" width="0" layer="19" extent="1-1"/>
-<wire x1="-13.97" y1="-11.43" x2="48.34" y2="7.62" width="0" layer="19" extent="1-1"/>
+<wire x1="12.7" y1="19.05" x2="20.32" y2="11.43" width="0.381" layer="1"/>
 </signal>
 <signal name="VCC_2">
@@
 <wire x1="39.37" y1="64.77" x2="44.45" y2="64.77" width="0.381" layer="16"/>
 <contactref element="J1" pad="3"/>
-<wire x1="4.318" y1="43.434" x2="-8.89" y2="-11.43" width="0" layer="19" extent="1-1"/>
+<wire x1="12.7" y1="24.13" x2="4.318" y2="32.512" width="0.381" layer="1"/>
+<wire x1="4.318" y1="32.512" x2="4.318" y2="43.434" width="0.381" layer="1"/>
 </signal>
 <signal name="PHASE_A1">
@@
 <wire x1="19.66" y1="121.92" x2="21.59" y2="121.92" width="0.381" layer="1"/>
 <contactref element="J1" pad="5"/>
-<wire x1="-3.81" y1="-11.43" x2="32.766" y2="61.722" width="0" layer="19" extent="1-1"/>
+<wire x1="12.7" y1="29.21" x2="12.7" y2="43.18" width="0.381" layer="1"/>
+<wire x1="12.7" y1="43.18" x2="16.51" y2="46.99" width="0.381" layer="1"/>
+<wire x1="16.51" y1="46.99" x2="16.51" y2="55.88" width="0.381" layer="1"/>
+<wire x1="16.51" y1="55.88" x2="22.352" y2="61.722" width="0.381" layer="1"/>
+<wire x1="22.352" y1="61.722" x2="32.766" y2="61.722" width="0.381" layer="1"/>
 </signal>
 <signal name="COM1">
@@
 <wire x1="55.372" y1="59.182" x2="57.992" y2="59.182" width="0.381" layer="1"/>
 <wire x1="57.992" y1="59.182" x2="58.03" y2="59.22" width="0.381" layer="1"/>
-<wire x1="53.975" y1="92.075" x2="53.975" y2="91.44" width="0.381" layer="16"/>
-<wire x1="53.975" y1="91.44" x2="53.975" y2="70.993" width="0.381" layer="16"/>
-<wire x1="58.42" y1="66.548" x2="58.42" y2="64.77" width="0.381" layer="16"/>
+<wire x1="53.975" y1="92.075" x2="53.975" y2="74.803" width="0.381" layer="16"/>
+<wire x1="58.42" y1="70.358" x2="58.42" y2="64.77" width="0.381" layer="16"/>
 <wire x1="58.42" y1="64.77" x2="58.166" y2="64.516" width="0.381" layer="16"/>
 <wire x1="58.166" y1="64.516" x2="57.023" y2="64.516" width="0.381" layer="16"/>
@@
 <wire x1="54.229" y1="61.722" x2="54.229" y2="60.071" width="0.381" layer="16"/>
 <wire x1="54.229" y1="60.071" x2="55.118" y2="59.182" width="0.381" layer="16"/>
-<wire x1="53.975" y1="70.993" x2="58.42" y2="66.548" width="0.381" layer="16"/>
+<wire x1="53.975" y1="74.803" x2="58.42" y2="70.358" width="0.381" layer="16"/>
 </signal>
 <signal name="BH1">
@@
 <contactref element="DRIV3" pad="2"/>
 <wire x1="58.03" y1="60.82" x2="58.1089" y2="60.8989" width="0.381" layer="1"/>
-<wire x1="58.1089" y1="60.8989" x2="62.23" y2="60.8989" width="0.381" layer="1"/>
-<via x="62.23" y="60.8989" extent="1-16" drill="0.35"/>
-<wire x1="62.23" y1="60.8989" x2="66.1011" y2="60.8989" width="0.381" layer="16"/>
+<wire x1="58.1089" y1="60.8989" x2="64.77" y2="60.8989" width="0.381" layer="1"/>
+<via x="64.77" y="60.8989" extent="1-16" drill="0.35"/>
+<wire x1="64.77" y1="60.8989" x2="66.1011" y2="60.8989" width="0.381" layer="16"/>
 <wire x1="66.1011" y1="60.8989" x2="67.31" y2="59.69" width="0.381" layer="16"/>
 <wire x1="67.31" y1="59.69" x2="67.31" y2="59.182" width="0.381" layer="16"/>
@@
 <contactref element="J1" pad="4"/>
 <contactref element="STM1" pad="PA15"/>
-<wire x1="-6.35" y1="-11.43" x2="56.58" y2="65.47" width="0" layer="19" extent="1-1"/>
+<wire x1="12.7" y1="26.67" x2="10.16" y2="29.21" width="0.381" layer="1"/>
+<wire x1="10.16" y1="29.21" x2="10.16" y2="43.18" width="0.381" layer="1"/>
+<wire x1="10.16" y1="43.18" x2="12.7" y2="45.72" width="0.381" layer="1"/>
+<wire x1="12.7" y1="45.72" x2="12.7" y2="46.99" width="0.381" layer="1"/>
+<wire x1="12.7" y1="46.99" x2="11.43" y2="48.26" width="0.381" layer="1"/>
+<wire x1="11.43" y1="48.26" x2="11.43" y2="55.88" width="0.381" layer="1"/>
+<wire x1="25.4" y1="69.85" x2="36.83" y2="69.85" width="0.381" layer="1"/>
+<via x="36.83" y="69.85" extent="1-16" drill="0.35"/>
+<wire x1="11.43" y1="55.88" x2="25.4" y2="69.85" width="0.381" layer="1"/>
+<wire x1="36.83" y1="69.85" x2="40.64" y2="73.66" width="0.381" layer="16"/>
+<wire x1="56.515" y1="70.485" x2="56.515" y2="69.215" width="0.381" layer="16"/>
+<via x="56.515" y="69.215" extent="1-16" drill="0.35"/>
+<wire x1="56.515" y1="69.215" x2="56.58" y2="69.15" width="0.381" layer="1"/>
+<wire x1="56.58" y1="69.15" x2="56.58" y2="65.47" width="0.381" layer="1"/>
+<wire x1="40.64" y1="73.66" x2="53.34" y2="73.66" width="0.381" layer="16"/>
+<wire x1="53.34" y1="73.66" x2="56.515" y2="70.485" width="0.381" layer="16"/>
 </signal>
 <signal name="SWCLK">
 <contactref element="J1" pad="2"/>
 <contactref element="STM1" pad="PA14"/>
-<wire x1="-11.43" y1="-11.43" x2="58.03" y2="64.02" width="0" layer="19" extent="1-1"/>
+<wire x1="12.7" y1="21.59" x2="17.78" y2="21.59" width="0.381" layer="1"/>
+<via x="17.78" y="21.59" extent="1-16" drill="0.35"/>
+<wire x1="17.78" y1="21.59" x2="25.4" y2="21.59" width="0.381" layer="16"/>
+<via x="25.4" y="21.59" extent="1-16" drill="0.35"/>
+<wire x1="25.4" y1="21.59" x2="30.48" y2="26.67" width="0.381" layer="1"/>
+<wire x1="30.48" y1="26.67" x2="49.53" y2="26.67" width="0.381" layer="1"/>
+<wire x1="49.53" y1="26.67" x2="53.34" y2="30.48" width="0.381" layer="1"/>
+<wire x1="53.34" y1="30.48" x2="55.88" y2="30.48" width="0.381" layer="1"/>
+<wire x1="55.88" y1="30.48" x2="57.15" y2="31.75" width="0.381" layer="1"/>
+<wire x1="57.15" y1="31.75" x2="57.15" y2="33.02" width="0.381" layer="1"/>
+<via x="57.15" y="33.02" extent="1-16" drill="0.35"/>
+<wire x1="57.15" y1="33.02" x2="57.15" y2="50.8" width="0.381" layer="16"/>
+<wire x1="57.15" y1="50.8" x2="63.5" y2="57.15" width="0.381" layer="16"/>
+<via x="63.5" y="63.5" extent="1-16" drill="0.35"/>
+<wire x1="63.5" y1="57.15" x2="63.5" y2="63.5" width="0.381" layer="16"/>
+<wire x1="58.03" y1="64.02" x2="58.042" y2="64.008" width="0.381" layer="1"/>
+<wire x1="62.992" y1="64.008" x2="63.5" y2="63.5" width="0.381" layer="1"/>
+<wire x1="58.042" y1="64.008" x2="62.992" y2="64.008" width="0.381" layer="1"/>
 </signal>
 </signals>

Commit message: done
Routing:
- net VCC_2: track 454.7 -> 463.6 mm
- net PWM_IN: track 83.5 -> 78.9 mm
Changed lines of the file:
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@@
 <drawing>
 <settings>
-<setting alwaysvectorfont="no"/>
+<setting alwaysvectorfont="yes"/>
 <setting verticaltext="up"/>
 </settings>
@@
 <wire x1="41.91" y1="116.84" x2="41.91" y2="106.68" width="0.762" layer="16"/>
 <wire x1="41.91" y1="106.68" x2="33.02" y2="97.79" width="0.762" layer="16"/>
-<via x="20.32" y="97.79" extent="1-16" drill="0.35" diameter="1.05"/>
+<via x="20.32" y="97.79" extent="1-16" drill="0.35" diameter="1.3"/>
 <wire x1="20.32" y1="97.79" x2="8.89" y2="97.79" width="0.762" layer="1"/>
 <wire x1="8.89" y1="97.79" x2="7.62" y2="96.52" width="0.762" layer="1"/>
 <wire x1="7.62" y1="81.28" x2="11.43" y2="77.47" width="0.762" layer="1"/>
-<wire x1="11.43" y1="77.47" x2="11.43" y2="73.66" width="0.762" layer="1"/>
-<wire x1="9.144" y1="71.374" x2="6.858" y2="71.374" width="0.762" layer="1"/>
+<wire x1="11.43" y1="77.47" x2="11.43" y2="71.12" width="0.762" layer="1"/>
 <wire x1="33.02" y1="97.79" x2="20.32" y2="97.79" width="0.762" layer="16"/>
 <wire x1="7.62" y1="96.52" x2="7.62" y2="81.28" width="0.762" layer="1"/>
-<wire x1="11.43" y1="73.66" x2="9.144" y2="71.374" width="0.762" layer="1"/>
 <polygon width="0.762" layer="1" isolate="1.27">
-<vertex x="2.54" y="71.12"/>
-<vertex x="8.89" y="71.12"/>
+<vertex x="3.81" y="72.39"/>
+<vertex x="7.62" y="72.39"/>
 <vertex x="9.398" y="70.612"/>
 <vertex x="9.398" y="58.801"/>
@@
 <wire x1="87.63" y1="95.25" x2="86.36" y2="96.52" width="1.016" layer="1"/>
 <wire x1="86.36" y1="96.52" x2="86.36" y2="100.33" width="1.016" layer="1"/>
+<wire x1="6.858" y1="66.548" x2="6.858" y2="61.214" width="0.762" layer="1"/>
+<wire x1="11.43" y1="71.12" x2="6.858" y2="66.548" width="0.762" layer="1"/>
 </signal>
 <signal name="GND">
@@
 <contactref element="STM1" pad="PA6"/>
 <contactref element="JP1" pad="1"/>
-<wire x1="53.34" y1="7.62" x2="53.34" y2="26.67" width="0.381" layer="16"/>
+<wire x1="54.737" y1="8.763" x2="53.594" y2="7.62" width="0.381" layer="16"/>
+<wire x1="53.34" y1="7.62" x2="53.594" y2="7.62" width="0.381" layer="16"/>
 <via x="54.737" y="53.467" extent="1-16" drill="0.35"/>
 <wire x1="53.38" y1="56.97" x2="53.38" y2="54.824" width="0.381" layer="1"/>
 <wire x1="53.38" y1="54.824" x2="54.737" y2="53.467" width="0.381" layer="1"/>
-<wire x1="54.737" y1="28.067" x2="54.737" y2="53.467" width="0.381" layer="16"/>
-<wire x1="53.34" y1="26.67" x2="54.737" y2="28.067" width="0.381" layer="16"/>
-<wire x1="26.67" y1="11.43" x2="39.37" y2="24.13" width="0.381" layer="16"/>
-<wire x1="39.37" y1="24.13" x2="50.8" y2="24.13" width="0.381" layer="16"/>
-<wire x1="50.8" y1="24.13" x2="53.34" y2="26.67" width="0.381" layer="16"/>
+<wire x1="54.737" y1="8.763" x2="54.737" y2="53.467" width="0.381" layer="16"/>
+<wire x1="26.67" y1="11.43" x2="49.53" y2="11.43" width="0.762" layer="1"/>
+<wire x1="49.53" y1="11.43" x2="53.34" y2="7.62" width="0.762" layer="1"/>
 </signal>
 <signal name="TEST_LED4">
